File: unoshield-v2.brd (EAGLE design)
At the start: 54.6 x 63.5 mm, 25 parts, among them Q1 FDS5680, X1 SPRING-TERMINAL, X2 SPRING-TERMINAL

Commit message: uno shield design work
Parts:
- removed JP2, JP6, JP7: M01PTH, SparkFun-Connectors:1X01
- added J3: (no value), SparkFun-Connectors:1X06
- added J4: 455-1750-1-ND, SparkFun-Connectors:1X03
- moved J2 36.0 mm to (10.2, 1.91)
Connections:
- new net N$14: J3.5, U$1.A3
- net 5V: now also J3.2, J4.3; no longer JP7.1
- net CL: now also J3.3
- net DA: now also J3.4
- net GND: now also J1.1, J3.1, J4.1; no longer J1.5, JP6.1
- net N$10: now also J1.4; no longer J1.3
- net N$11: now also J1.5; no longer J1.4
- net N$28: now also J3.6
- net N$6: now also J4.2; no longer JP2.1
- net N$7: now also J1.2; no longer J1.1
- net N$9: now also J1.3; no longer J1.2
Routing:
- net N$13: track 0.00 -> 31.4 mm
- net 5V: track 48.2 -> 67.4 mm
- net DA: track 17.0 -> 26.1 mm
- net CL: track 14.1 -> 23.3 mm
- net N$14: track 0.00 -> 9.12 mm
- net N$11: track 30.7 -> 28.2 mm
- net N$9: track 40.9 -> 38.4 mm
- net N$7: track 46.0 -> 43.4 mm
- net N$10: track 35.8 -> 33.3 mm
- net N$28: track 26.2 -> 28.2 mm
Other:
- board text added: "2.5 V"
- board text added: "5V"
- board text added: "A3"
- board text added: "A4"
- board text added: "A5"
- board text added: "D5"
- board text added: "D8"
- board text added: "EXT I/O"
- board text added: "PTV09A-4030U-B203-ND"
- board text added: "SSW-105-02-G-S SAM1209-05-ND"
- board text added: "UNO SHIELD V 2 PUBLIC DOMAIN MARCH 2019"
- board text removed: "PTV09A- 4030U -B203-ND"
- board text removed: "UNO SHIELD PUBLIC DOMAIN JANUARY 2019"
