File: unoshield-v2.sch (EAGLE design)
At the start: 19 parts, among them Q1 FDS5680, X1 SPRING-TERMINAL, X2 SPRING-TERMINAL

Commit message: uno shield design work
Parts:
- removed JP2, JP6, JP7: M01PTH, SparkFun-Connectors:M01PTH
- added J2: (no value), SparkFun-Connectors:CONN_02
- added J3: (no value), SparkFun-Connectors:CONN_06SILK_FEMALE_PTH
- added J4: 455-1750-1-ND, SparkFun-Connectors:CONN_03
- added JP10, JP11, JP12, JP8, JP9: M01PTH, SparkFun-Connectors:M01PTH
Connections:
- new net N$12: JP11.1, JP9.1, U$1.D2
- new net N$13: J2.1, U$1.D8
- new net N$14: J3.5, U$1.A3
- net 5V: now also J3.2, J4.3; no longer C1.+, JP5.2, JP7.1
- net BUTTON: now also JP10.1, U$1.*D3; no longer U$1.D2
- net CL: now also J3.3
- net DA: now also J3.4
- net GND: now also J1.1, J2.2, J3.1, J4.1, JP12.1, JP8.1; no longer J1.5, JP6.1
- net N$10: now also J1.4; no longer J1.3
- net N$11: now also J1.5; no longer J1.4
- net N$28: now also J3.6
- net N$6: now also J4.2; no longer JP2.1
- net N$7: now also J1.2; no longer J1.1
- net N$9: now also J1.3; no longer J1.2
- net VIN: now also C1.+, JP5.2
Other:
- moved on the sheet: J1
